File: pcb/dongle.kicad_pcb (KiCad board)
At the start: 2 copper layers, 23 parts, among them J1 USB_A, J2 Conn_01x01_Pin, J3 Conn_01x01_Pin, J4 Conn_01x01_Pin, J5 Conn_01x01_Pin, U3 nRF52833_QDxx, Y1 32MHz

Commit message: update pcb
Parts:
- added D1: BLUE, dongle:LED_0603_1608Metric, F.Cu at (167.7, 102.4)
- added R1: 1K, dongle:R_0201_0603Metric_Pad0.64x0.40mm_HandSolder, F.Cu at (167.7, 99.6)
- added SW1: SW_Push_45deg, dongle:TS342A2P, F.Cu at (162.7, 96.8)
- moved U3 28.5 mm to (159.1, 102.3)
- moved AE1 25.2 mm to (169.1, 107.5), turned to -90 degrees
- moved Y1 24.2 mm to (165.1, 100.9)
- moved C13 21.1 mm to (158.5, 97.8), turned to -90 degrees
- moved C12 19.1 mm to (157.3, 97.8), turned to -90 degrees
- moved C4 18.3 mm to (165.1, 104.1), turned to 90 degrees
- moved C2 17.8 mm to (165.7, 102.5)
- moved C1 17.5 mm to (164.5, 99.3)
- moved C3 16.2 mm to (163.7, 104.1), turned to 90 degrees
- moved C5 16.0 mm to (154.9, 100.9), turned to 90 degrees
- moved L2 15.9 mm to (166.9, 107.0)
- moved L1 15.9 mm to (166.9, 105.3)
- moved C7 15.4 mm to (159.7, 105.9)
- moved C11 14.8 mm to (162.7, 99.9), turned to -90 degrees
- moved J2 14.6 mm to (157.9, 109.2), turned to 90 degrees
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Connections:
- AE1 pad 2: VSS -> (no net)
- U3 pad 23: unconnected-(U3-NFC2/P0.10-Pad23) -> LED
Other:
- board outline added: 30.2 x 15.5 mm

Commit message: update pcb
Parts:
- removed SW1: SW_Push_45deg, dongle:TS342A2P
- AE1: value Antenna -> Antenna_Shield; footprint dongle:Texas_SWRA117D_2.4GHz_Left -> dongle:ANTC5020X110N
- C1, C10, C11, C2, C3, C4, C5, C7: footprint dongle:C_0201_0603Metric_Pad0.64x0.40mm_HandSolder -> dongle:C_0201_0603Metric
- C12, C13: footprint dongle:C_0402_1005Metric_Pad0.74x0.62mm_HandSolder -> dongle:C_0402_1005Metric
- C17, C19, C6: footprint dongle:C_0603_1608Metric_Pad1.08x0.95mm_HandSolder -> dongle:C_0603_1608Metric
- D1: footprint dongle:LED_0603_1608Metric -> dongle:LED_0402_1005Metric
- J2, J3, J4: footprint dongle:TestPoint_Pad_1.0x1.0mm -> dongle:TestPoint_Pad_D1.0mm
- J5: footprint dongle:TestPoint_Pad_D1.0mm -> dongle:TestPoint_Pad_1.0x1.0mm
- L1, L2: footprint dongle:L_0201_0603Metric_Pad0.64x0.40mm_HandSolder -> dongle:L_0201_0603Metric
- R1: footprint dongle:R_0201_0603Metric_Pad0.64x0.40mm_HandSolder -> dongle:R_0402_1005Metric
- Y1: value 32MHz -> Crystal_GND24; footprint dongle:Crystal_SMD_2012-2Pin_2.0x1.2mm_HandSoldering -> dongle:Crystal_SMD_3225-4Pin_3.2x2.5mm
- moved R1 42.8 mm to (153.1, 139.8), turned to 0 degrees
- moved C1 42.5 mm to (161.3, 141.7), turned to -90 degrees
- moved C11 41.8 mm to (160.1, 141.6), turned to 90 degrees
- moved D1 41.2 mm to (153.1, 140.9), turned to 0 degrees
- moved AE1 40.1 mm to (154.0, 144.7), turned to 0 degrees
- moved Y1 39.7 mm to (163.8, 140.6)
- moved C10 39.4 mm to (158.9, 141.5)
- moved C13 39.2 mm to (162.4, 136.9), turned to 180 degrees
- moved C4 38.7 mm to (155.4, 141.6), turned to -90 degrees
- moved C12 38.4 mm to (162.4, 135.9), turned to 180 degrees
- moved C3 37.9 mm to (157.7, 141.6)
- moved L1 37.4 mm to (156.5, 141.3), turned to 180 degrees
- moved L2 36.7 mm to (154.5, 141.6), turned to -90 degrees
- moved C2 35.8 mm to (164.6, 138.3)
- moved U3 35.4 mm to (158.3, 137.7), turned to -90 degrees
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Connections:
- AE1 pad 1: Net-(AE1-A) -> unconnected-(AE1-A-Pad1)
- AE1 pad 2: (no net) -> Net-(AE1-Shield)
- C1 pad 1: XC2 -> VSS
- C1 pad 2: VSS -> XC1
- C2 pad 2: XC1 -> XC2
- L2 pad 2: Net-(AE1-A) -> Net-(AE1-Shield)
- Y1 pad 1: XC2 -> XC1
- Y1 pad 2: XC1 -> VSS
Routing:
- net D+: track 0.00 -> 17.1 mm
- net XC2: track 0.00 -> 10.6 mm
- net D-: track 0.00 -> 10.2 mm
- net VDD: track 0.00 -> 6.30 mm, vias 0 -> 1
- net XC1: track 0.00 -> 6.04 mm
- net LED: track 0.00 -> 4.30 mm
- net Net-(AE1-Shield): track 0.00 -> 3.49 mm
- net SWD: track 0.00 -> 3.35 mm, vias 0 -> 1
- net ANT: track 0.00 -> 2.00 mm
- net SWC: track 0.00 -> 1.81 mm, vias 0 -> 1
- net DECUSB: track 0.00 -> 1.77 mm
- net Net-(C4-Pad1): track 0.00 -> 1.70 mm
- net VBUS: track 0.00 -> 1.68 mm
- net Net-(D1-K): track 0.00 -> 1.47 mm
- net DEC4: track 0.00 -> 1.28 mm
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- added copper zone on B.Cu, net VSS
- added copper zone on F.Cu, net VSS
Other:
- board size 30.2 x 15.5 mm -> 15.5 x 20.1 mm

Commit message: udpate footprint
Parts:
- added C15: 7pF, dongle:C_0201_0603Metric, F.Cu at (174.0, 134.9)
- added C16: 7pF, dongle:C_0201_0603Metric, F.Cu at (174.0, 136.7)
- added Y2: Crystal_Small, dongle:Crystal_SMD_3215-2Pin_3.2x1.5mm, F.Cu at (182.7, 139.2)
- AE1: footprint dongle:ANTC5020X110N -> dongle:AN9520-245
- J1: moved to B.Cu
- Y1: footprint dongle:Crystal_SMD_3225-4Pin_3.2x2.5mm -> dongle:Crystal_SMD_2520-4Pin_2.5x2.0mm
- moved J3 43.7 mm to (192.2, 118.1)
- moved J4 43.7 mm to (192.2, 120.1)
- moved R1 39.2 mm to (192.0, 135.3)
- moved D1 36.4 mm to (189.1, 135.3)
- moved J2 35.3 mm to (192.2, 116.1)
- moved J5 30.8 mm to (192.2, 122.1)
- moved Y1 27.2 mm to (189.7, 132.3)
- moved C13 26.5 mm to (188.9, 139.3), turned to 0 degrees
- moved C12 26.4 mm to (188.9, 137.3), turned to 0 degrees
- moved C19 23.4 mm to (177.3, 140.3), turned to 0 degrees
- moved C17 22.5 mm to (177.3, 137.8)
- moved L2 19.6 mm to (174.0, 140.2), turned to 0 degrees
- moved C6 19.2 mm to (177.3, 135.3), turned to 0 degrees
- moved L1 17.7 mm to (174.0, 138.4), turned to 0 degrees
- moved C7 17.3 mm to (171.6, 136.7)
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Routing:
- net D+: track 17.1 -> 0.00 mm
- net XC2: track 10.6 -> 0.00 mm
- net D-: track 10.2 -> 0.00 mm
- net VDD: track 6.30 -> 0.00 mm, vias 1 -> 0
- net XC1: track 6.04 -> 0.00 mm
- net LED: track 4.30 -> 0.00 mm
- net Net-(AE1-Shield): track 3.49 -> 0.00 mm
- net SWD: track 3.35 -> 0.00 mm, vias 1 -> 0
- net ANT: track 2.00 -> 0.00 mm
- net SWC: track 1.81 -> 0.00 mm, vias 1 -> 0
- net DECUSB: track 1.77 -> 0.00 mm
- net Net-(C4-Pad1): track 1.70 -> 0.00 mm
- net VBUS: track 1.68 -> 0.00 mm
- net Net-(D1-K): track 1.47 -> 0.00 mm
- net DEC4: track 1.28 -> 0.00 mm
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- removed copper zone on B.Cu, net VSS
- removed copper zone on F.Cu, net VSS

Commit message: upload v0.1
Parts:
- added SW1: SW_Push_45deg, dongle:SW_SPST_B3U-1000P, B.Cu at (146.6, 108.9)
- D1, R1: moved to B.Cu
- J1: footprint dongle:USB_A_Connfly_DS1098_Horizontal -> dongle:USB_A_Molex_48037-2200_Horizontal; moved to F.Cu
- moved R1 58.4 mm to (140.7, 107.5), turned to 180 degrees
- moved D1 56.4 mm to (140.7, 106.5), turned to 180 degrees
- moved J4 53.5 mm to (140.8, 105.1)
- moved C19 53.4 mm to (140.8, 101.2)
- moved C13 52.8 mm to (150.4, 103.1), turned to 90 degrees
- moved C12 52.5 mm to (149.4, 102.6), turned to 90 degrees
- moved J2 51.7 mm to (141.9, 103.8)
- moved J3 49.9 mm to (143.3, 107.9)
- moved C6 49.4 mm to (143.5, 99.2), turned to -90 degrees
- moved Y1 48.4 mm to (147.1, 109.3)
- moved C17 47.5 mm to (150.0, 98.8), turned to 180 degrees
- moved Y2 46.4 mm to (150.2, 106.1), turned to -90 degrees
- moved J5 46.0 mm to (151.7, 100.3)
- moved L2 44.1 mm to (141.5, 110.3), turned to 180 degrees
- moved C7 43.2 mm to (141.9, 105.2), turned to 90 degrees
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Connections:
- AE1 pad 1: unconnected-(AE1-A-Pad1) -> Net-(AE1-A)
- AE1 pad 2: Net-(AE1-Shield) -> unconnected-(AE1-Shield-Pad2)
- L2 pad 2: Net-(AE1-Shield) -> Net-(AE1-A)
Routing:
- net RESET: track 0.00 -> 14.4 mm, vias 0 -> 1
- net XL2: track 0.00 -> 13.7 mm
- net D-: track 0.00 -> 13.0 mm, vias 0 -> 1
- net VBUS: track 0.00 -> 9.92 mm, vias 0 -> 1
- net XL1: track 0.00 -> 9.50 mm
- net D+: track 0.00 -> 9.35 mm, vias 0 -> 1
- net VDD: track 0.00 -> 6.94 mm, vias 0 -> 2
- net XC1: track 0.00 -> 5.82 mm
- net LED: track 0.00 -> 5.28 mm, vias 0 -> 1
- net XC2: track 0.00 -> 3.85 mm
- net ANT: track 0.00 -> 3.76 mm
- net VSS: track 0.00 -> 3.33 mm, vias 0 -> 7
- net SWD: track 0.00 -> 3.18 mm, vias 0 -> 1
- net DEC4: track 0.00 -> 2.26 mm
- net SWC: track 0.00 -> 2.21 mm, vias 0 -> 2
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- added copper zone on B.Cu, net VSS
- added copper zone on F.Cu, net VSS
Other:
- board size 15.5 x 20.1 mm -> 14 x 20 mm
- board text added: "SWC"
- board text added: "SWD"
- board text added: "VDD"
- board text added: "VSS"

Commit message: clear pcb
Parts:
- D1, R1, SW1: moved to F.Cu
- moved R1 21.4 mm to (160.1, 116.5), turned to 0 degrees
- moved D1 21.2 mm to (160.3, 114.5), turned to 0 degrees
- moved J1 20.8 mm to (143.7, 109.9)
- moved Y2 19.0 mm to (159.7, 122.5), turned to 0 degrees
- moved U3 16.1 mm to (155.0, 117.2), turned to 0 degrees
- moved L2 16.1 mm to (157.5, 112.7), turned to 0 degrees
- moved SW1 16.0 mm to (154.3, 123.0), turned to 0 degrees
- moved Y1 15.3 mm to (159.6, 100.6)
- moved C19 15.0 mm to (155.3, 104.8)
- moved L1 13.9 mm to (157.5, 110.9), turned to 0 degrees
- moved C7 13.7 mm to (155.0, 109.2), turned to 0 degrees
- moved AE1 12.1 mm to (140.5, 123.8)
- moved C6 11.9 mm to (155.3, 99.8), turned to 0 degrees
- moved J4 11.7 mm to (152.3, 103.5)
- moved J2 11.3 mm to (152.3, 99.5)
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Connections:
- C1 pad 1: VSS -> GND
- C10 pad 1: VSS -> GND
- C11 pad 1: VSS -> GND
- C12 pad 1: VSS -> GND
- C13 pad 1: VSS -> GND
- C15 pad 2: VSS -> GND
- C16 pad 1: VSS -> GND
- C17 pad 1: VSS -> GND
- C19 pad 1: VSS -> GND
- C2 pad 1: VSS -> GND
- C3 pad 1: VSS -> VSS_PA
- C4 pad 2: VSS -> GND
- C5 pad 1: VSS -> GND
- C6 pad 1: VSS -> GND
- C7 pad 1: VSS -> GND
- J1 pad 4: VSS -> GND
- J1 pad 5: VSS -> GND
- J5 pad 1: VSS -> GND
- R1 pad 2: VSS -> GND
- SW1 pad 2: VSS -> GND
- U3 pad 25: VSS -> VSS_PA
- U3 pad 37: VSS -> GND
- U3 pad 41: VSS -> GND
- Y1 pad 2: VSS -> GND
- Y1 pad 4: VSS -> GND
Routing:
- net RESET: track 14.4 -> 0.00 mm, vias 1 -> 0
- net XL2: track 13.7 -> 0.00 mm
- net D-: track 13.0 -> 0.00 mm, vias 1 -> 0
- net VBUS: track 9.92 -> 0.00 mm, vias 1 -> 0
- net XL1: track 9.50 -> 0.00 mm
- net D+: track 9.35 -> 0.00 mm, vias 1 -> 0
- net VDD: track 6.94 -> 0.00 mm, vias 2 -> 0
- net XC1: track 5.82 -> 0.00 mm
- net LED: track 5.28 -> 0.00 mm, vias 1 -> 0
- net XC2: track 3.85 -> 0.00 mm
- net ANT: track 3.76 -> 0.00 mm
- net VSS: track 3.33 -> 0.00 mm, vias 7 -> 0
- net SWD: track 3.18 -> 0.00 mm, vias 1 -> 0
- net DEC4: track 2.26 -> 0.00 mm
- net SWC: track 2.21 -> 0.00 mm, vias 2 -> 0
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- removed copper zone on B.Cu, net VSS
- removed copper zone on F.Cu, net VSS
Other:
- board outline removed
- board text removed: "SWC"
- board text removed: "SWD"
- board text removed: "VDD"
- board text removed: "VSS"

Commit message: update pcb
Parts:
- added REF**: MountingHole_1.1mm, dongle:MountingHole_1.1mm, F.Cu at (188.8, 120.5)
- added REF**: MountingHole_1.1mm, dongle:MountingHole_1.1mm, F.Cu at (177.2, 120.5)
- D1, R1, SW1: moved to B.Cu
- moved AE1 41.6 mm to (181.4, 131.7)
- moved C1 39.8 mm to (189.1, 123.3), turned to -90 degrees
- moved C2 39.6 mm to (187.6, 127.6), turned to 180 degrees
- moved J1 39.2 mm to (182.9, 110.3)
- moved Y1 38.0 mm to (188.2, 125.6), turned to 180 degrees
- moved J3 37.4 mm to (179.8, 126.8)
- moved J2 36.0 mm to (178.2, 124.5)
- moved C17 35.6 mm to (186.5, 119.5), turned to -90 degrees
- moved C12 35.0 mm to (188.5, 122.0), turned to 180 degrees
- moved C5 34.8 mm to (186.7, 121.8), turned to 180 degrees
- moved C11 34.6 mm to (186.3, 127.5), turned to -90 degrees
- moved C3 34.5 mm to (182.4, 128.2), turned to 180 degrees
- moved SW1 34.1 mm to (188.2, 126.7), turned to -90 degrees
- moved C10 33.8 mm to (184.0, 128.3), turned to 135 degrees
- moved C13 33.5 mm to (187.2, 123.2), turned to 180 degrees
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Connections:
- C13 pad 2: DEC4 -> DEC4_6
- U3 pad 21: DEC5 -> unconnected-(U3-DEC5-Pad21)
- U3 pad 26: DEC6 -> DEC4_6
- U3 pad 38: DEC4 -> DEC4_6
Routing:
- net DEC4_6: track 0.00 -> 16.6 mm, vias 0 -> 2
- net D-: track 0.00 -> 15.9 mm, vias 0 -> 1
- net RESET: track 0.00 -> 12.3 mm, vias 0 -> 1
- net D+: track 0.00 -> 11.3 mm, vias 0 -> 1
- net XC1: track 0.00 -> 11.1 mm
- net VDD: track 0.00 -> 9.71 mm, vias 0 -> 1
- net VBUS: track 0.00 -> 9.59 mm, vias 0 -> 1
- net XC2: track 0.00 -> 5.16 mm
- net SWD: track 0.00 -> 3.96 mm, vias 0 -> 1
- net Net-(AE1-A): track 0.00 -> 3.82 mm
- net XL2: track 0.00 -> 3.81 mm
- net LED: track 0.00 -> 3.68 mm, vias 0 -> 1
- net XL1: track 0.00 -> 3.14 mm
- net DECUSB: track 0.00 -> 2.35 mm
- net ANT: track 0.00 -> 2.17 mm
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- added copper zone on B.Cu, net GND
- added copper zone on F.Cu, net GND
Other:
- board outline added: 14 x 18.1 mm

Commit message: update pcb
Parts:
- removed REF** (x2): MountingHole_1.1mm, dongle:MountingHole_1.1mm
- removed SW1: SW_Push_45deg, dongle:SW_SPST_B3U-1000P
- D1, R1: moved to F.Cu
- J1: footprint dongle:USB_A_Molex_48037-2200_Horizontal -> dongle:USB_A_PCB_Edge_receptacle
- U3: footprint dongle:QFN-40-1EP_5x5mm_P0.4mm_EP3.6x3.6mm_ThermalVias -> dongle:QFN-40-1EP_5x5mm_P0.4mm_EP3.6x3.6mm
- moved C17 53.8 mm to (142.9, 88.0)
- moved C19 51.2 mm to (142.9, 84.8), turned to -90 degrees
- moved C2 51.1 mm to (152.2, 90.8)
- moved C11 50.6 mm to (152.2, 90.1), turned to 180 degrees
- moved C6 50.5 mm to (144.4, 84.8)
- moved C12 50.3 mm to (152.3, 87.1)
- moved C5 49.9 mm to (151.8, 86.2)
- moved U3 49.9 mm to (148.2, 88.8)
- moved C15 49.9 mm to (146.7, 83.8), turned to 180 degrees
- moved C10 49.6 mm to (149.4, 92.8)
- moved C7 49.5 mm to (144.3, 90.3), turned to 45 degrees
- moved C13 49.5 mm to (152.3, 88.1)
- moved Y2 49.4 mm to (149.4, 84.5)
- moved AE1 49.3 mm to (146.3, 97.0)
- moved C3 48.9 mm to (148.1, 93.3)
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Routing:
- net GND: track 0.00 -> 16.4 mm, vias 12 -> 3
- net D-: track 15.9 -> 0.00 mm, vias 1 -> 0
- net RESET: track 12.3 -> 0.00 mm, vias 1 -> 0
- net D+: track 11.3 -> 0.00 mm, vias 1 -> 0
- net XC1: track 11.1 -> 6.73 mm
- net VDD: track 9.71 -> 12.9 mm
- net VBUS: track 9.59 -> 7.15 mm, vias 1 -> 2
- net LED: track 3.68 -> 1.52 mm
- net VSS_PA: track 0.95 -> 2.21 mm
- net XC2: track 5.16 -> 4.08 mm
- net DECUSB: track 2.35 -> 3.40 mm
- net SWC: track 1.00 -> 1.94 mm
- net ANT: track 2.17 -> 2.86 mm
- net DEC4_6: track 16.6 -> 17.3 mm, vias 2 -> 0
- net Net-(AE1-A): track 3.82 -> 4.44 mm
Other:
- board size 14 x 18.1 mm -> 12 x 15 mm

Commit message: update footprint
Parts:
- J1: footprint dongle:USB_A_PCB_Edge_receptacle -> dongle:USB_A_PCB_Edge
- J2, J3, J4: footprint dongle:TestPoint_Pad_D1.0mm -> dongle:TestPoint_Pad_R
- J5: footprint dongle:TestPoint_Pad_1.0x1.0mm -> dongle:TestPoint_Pad
- moved Y2 34.6 mm to (167.0, 114.3), turned to 0 degrees
- moved R1 31.7 mm to (171.0, 113.7)
- moved C15 28.8 mm to (158.3, 110.0), turned to 0 degrees
- moved U3 28.4 mm to (168.1, 109.0), turned to 0 degrees
- moved C19 28.1 mm to (167.3, 98.8), turned to 0 degrees
- moved J5 27.9 mm to (170.2, 98.9)
- moved C16 27.7 mm to (158.3, 111.8), turned to 0 degrees
- moved J2 26.2 mm to (170.2, 93.5)
- moved C17 25.7 mm to (167.3, 96.3), turned to 0 degrees
- moved D1 25.7 mm to (161.2, 114.1), turned to 0 degrees
- moved C13 25.5 mm to (161.0, 112.1), turned to 0 degrees
- moved C11 25.5 mm to (155.9, 115.3), turned to 0 degrees
- moved J4 25.3 mm to (170.2, 97.1)
- moved C12 24.6 mm to (161.0, 110.2), turned to 0 degrees
- moved C6 24.6 mm to (167.3, 93.8), turned to 0 degrees
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Connections:
- C13 pad 2: DEC4_6 -> DEC4
- U3 pad 26: DEC4_6 -> unconnected-(U3-DEC6-Pad26)
- U3 pad 38: DEC4_6 -> DEC4
Routing:
- net DEC4_6: track 17.3 -> 0.00 mm
- net GND: track 16.4 -> 0.00 mm, vias 3 -> 0
- net VDD: track 12.9 -> 0.00 mm, vias 1 -> 0
- net VBUS: track 7.15 -> 0.00 mm, vias 2 -> 0
- net XC1: track 6.73 -> 0.00 mm
- net Net-(AE1-A): track 4.44 -> 0.00 mm
- net XC2: track 4.08 -> 0.00 mm
- net XL2: track 3.79 -> 0.00 mm
- net SWD: track 3.75 -> 0.00 mm, vias 1 -> 0
- net XL1: track 3.47 -> 0.00 mm
- net DECUSB: track 3.40 -> 0.00 mm
- net ANT: track 2.86 -> 0.00 mm
- net VSS_PA: track 2.21 -> 0.00 mm
- net SWC: track 1.94 -> 0.00 mm, vias 1 -> 0
- net Net-(C4-Pad1): track 1.55 -> 0.00 mm
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Other:
- board size 12 x 15 mm -> 12 x 16 mm
