File: pcb/dongle.kicad_pcb (KiCad board)
At the start: 2 copper layers, 12 x 17.6 mm, 29 parts, among them J1 USB_A, J2 Conn_01x01_Pin, J3 Conn_01x01_Pin, J4 Conn_01x01_Pin, J5 Conn_01x01_Pin, SW1 SW_Push_45deg, U3 nRF52833_QDxx, Y1 Crystal_GND24, Y2 Crystal_Small

Commit message: update ibom
Parts:
- C15, C16: value 7pF -> 12pF
Changed lines of the file:
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@@
 			)
 		)
-		(property "Value" "7pF"
+		(property "Value" "12pF"
 			(at 0 1.05 90)
 			(layer "F.Fab")
@@
 			)
 		)
-		(property "JLCPCB" "C276424"
+		(property "JLCPCB" "C5213671"
 			(at 0 0 0)
 			(layer "F.SilkS")
@@
 			)
 		)
-		(property "Value" "7pF"
+		(property "Value" "12pF"
 			(at 0 1.05 90)
 			(layer "F.Fab")
@@
 		(layer "Edge.Cuts")
 	)
+	(dimension
+		(type orthogonal)
+		(layer "Dwgs.User")
+		(pts
+			(xy 150 92.035) (xy 150 80.035)
+		)
+		(height -1.93)
+		(orientation 1)
+		(format
+			(prefix "")
+			(suffix "")
+			(units 3)
+			(units_format 0)
+			(precision 4)
+			(suppress_zeroes yes)
+		)
+		(style
+			(thickness 0.1)
+			(arrow_length 1.27)
+			(text_position_mode 2)
+			(arrow_direction outward)
+			(extension_height 0.58642)
+			(extension_offset 0.5)
+			(keep_text_aligned yes)
+		)
+		(gr_text "12"
+			(at 147.97 85.3 90)
+			(layer "Dwgs.User")
+			(effects
+				(font
+					(size 1 1)
+					(thickness 0.15)
+				)
+			)
+		)
+	)
+	(dimension
+		(type orthogonal)
+		(layer "Dwgs.User")
+		(pts
+			(xy 162 80.01) (xy 162 97.61)
+		)
+		(height 1.88)
+		(orientation 1)
+		(format
+			(prefix "")
+			(suffix "")
+			(units 3)
+			(units_format 0)
+			(precision 4)
+			(suppress_zeroes yes)
+		)
+		(style
+			(thickness 0.1)
+			(arrow_length 1.27)
+			(text_position_mode 2)
+			(arrow_direction outward)
+			(extension_height 0.58642)
+			(extension_offset 0.5)
+			(keep_text_aligned yes)
+		)
+		(gr_text "17.6"
+			(at 164 88.69 90)
+			(layer "Dwgs.User")
+			(effects
+				(font
+					(size 1 1)
+					(thickness 0.15)
+				)
+			)
+		)
+	)
 	(via

Commit message: try fix impedance
Routing:
- net GND: vias 36 -> 41
Changed lines of the file:
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@@
 	(generator_version "9.0")
 	(general
-		(thickness 1.6062)
+		(thickness 1.6)
 		(legacy_teardrops no)
 	)
@@
 				(type "core")
 				(color "FR4 natural")
-				(thickness 1.5162)
+				(thickness 1.51)
 				(material "7628")
 				(epsilon_r 4.5)
@@
 			(drillshape 0)
 			(scaleselection 1)
-			(outputdirectory "../../../../../dongle_gerber/")
+			(outputdirectory "../../../../../inpudongle/")
 		)
 	)
@@
 		(sheetfile "dongle.kicad_sch")
 		(attr exclude_from_pos_files)
-		(fp_text user "SWD"
+		(fp_text user "${REFERENCE}"
 			(at 0 0.55 0)
-			(layer "F.SilkS")
+			(layer "F.Fab")
 			(effects
 				(font
@@
 		(sheetfile "dongle.kicad_sch")
 		(attr exclude_from_pos_files)
-		(fp_text user "VDD"
-			(at 0 0.56 0)
-			(layer "F.SilkS")
+		(fp_text user "${REFERENCE}"
+			(at 0 0.55 0)
+			(layer "F.Fab")
 			(effects
 				(font
@@
 		(layer "F.Cu")
 		(at 152.205 91.1 -90)
-		(descr "SMD2520/4, Crystal, 2.5x2.0mm package, SMD, generated with kicad-footprint-generator make_crystal.py, http://www.newxtal.com/UploadFiles/Images/2012-11-12-09-29-09-776.pdf")
 		(property "Reference" "Y1"
 			(at 0 -2.2 90)
@@
 			)
 		)
+		(property "LCSC Part #" "C5261121"
+			(at 0 0 270)
+			(layer "F.SilkS")
+			(hide yes)
+			(effects
+				(font
+					(size 1 1)
+					(thickness 0.1)
+				)
+			)
+		)
 		(property "JLCPCB" "C5213671"
 			(at 0 0 90)
@@
 		(sheetfile "dongle.kicad_sch")
 		(attr exclude_from_pos_files)
-		(fp_text user "GND"
+		(fp_text user "${REFERENCE}"
 			(at 0 0.57 0)
-			(layer "F.SilkS")
+			(layer "F.Fab")
 			(effects
 				(font
@@
 		(sheetfile "dongle.kicad_sch")
 		(attr smd)
-		(fp_line
-			(start -0.153641 -0.38)
-			(end 0.153641 -0.38)
-			(stroke
-				(width 0.12)
-				(type solid)
-			)
-			(layer "F.SilkS")
-		)
-		(fp_line
-			(start -0.153641 0.38)
-			(end 0.153641 0.38)
-			(stroke
-				(width 0.12)
-				(type solid)
-			)
-			(layer "F.SilkS")
-		)
 		(fp_rect
 			(start -0.93 -0.47)
@@
 		(layer "F.Cu")
 		(at 153.88 81.62 180)
-		(descr "SMD Crystal FC-135 https://support.epson.biz/td/api/doc_check.php?dl=brief_FC-135R_en.pdf")
 		(tags "SMD SMT Crystal")
 		(property "Reference" "Y2"
@@
 			)
 		)
+		(property " LCSC Part #" "C5213671"
+			(at 0 0 180)
+			(layer "F.SilkS")
+			(hide yes)
+			(effects
+				(font
+					(size 1 1)
+					(thickness 0.1)
+				)
+			)
+		)
 		(property "JLCPCB" "C5213671"
 			(at 0 0 0)
@@
 		(sheetfile "dongle.kicad_sch")
 		(attr exclude_from_pos_files)
-		(fp_text user "SWC"
+		(fp_text user "${REFERENCE}"
 			(at 0 0.55 0)
-			(layer "F.SilkS")
+			(layer "F.Fab")
 			(effects
 				(font
@@
 		(attr smd)
 		(fp_line
-			(start -0.13 -0.25)
-			(end -0.13 0.25)
+			(start -0.875 -0.25)
+			(end -0.875 0.25)
 			(stroke
 				(width 0.1)
@@
 	)
 	(via
+		(at 160 94.55)
+		(size 0.5)
+		(drill 0.2)
+		(layers "F.Cu" "B.Cu")
+		(free yes)
+		(net 1)
+	)
+	(via
 		(at 160.98 85.93)
 		(size 0.5)
@@
 	)
 	(via
+		(at 161.3 93.28)
+		(size 0.5)
+		(drill 0.2)
+		(layers "F.Cu" "B.Cu")
+		(free yes)
+		(net 1)
+	)
+	(via
 		(at 150.38 86.62)
 		(size 0.5)
@@
 	)
 	(via
-		(at 151.28 94.36)
+		(at 160.38 80.37)
 		(size 0.5)
 		(drill 0.2)
@@
 	)
 	(via
-		(at 154.16 91.62)
+		(at 150.38 90.37)
 		(size 0.5)
 		(drill 0.2)
@@
 	)
 	(via
-		(at 160.38 80.37)
+		(at 161.63 89.12)
 		(size 0.5)
 		(drill 0.2)
@@
 	)
 	(via
-		(at 150.38 90.37)
+		(at 152.88 80.37)
 		(size 0.5)
 		(drill 0.2)
@@
 	)
 	(via
-		(at 161.63 89.12)
+		(at 150.38 91.62)
 		(size 0.5)
 		(drill 0.2)
@@
 	)
 	(via
-		(at 152.88 80.37)
+		(at 161.63 80.37)
 		(size 0.5)
 		(drill 0.2)
@@
 	)
 	(via
-		(at 155.085 91.62)
+		(at 150.4 92.76)
 		(size 0.5)
 		(drill 0.2)
@@
 	)
 	(via
-		(at 150.38 91.62)
+		(at 150.38 82.87)
 		(size 0.5)
 		(drill 0.2)
@@
 	)
 	(via
-		(at 161.63 80.37)
+		(at 154.13 80.37)
 		(size 0.5)
 		(drill 0.2)
@@
 	)
 	(via
-		(at 150.4 92.76)
+		(at 150.83 93.21)
 		(size 0.5)
 		(drill 0.2)
@@
 	)
 	(via
-		(at 150.38 82.87)
+		(at 150.38 81.62)
 		(size 0.5)
 		(drill 0.2)
@@
 	)
 	(via
-		(at 154.13 80.37)
+		(at 151.41 94.55)
 		(size 0.5)
 		(drill 0.2)
@@
 	)
 	(via
-		(at 150.83 93.21)
+		(at 150.38 87.87)
 		(size 0.5)
 		(drill 0.2)
@@
 	)
 	(via
-		(at 150.38 81.62)
+		(at 153.183333 94.55)
 		(size 0.5)
 		(drill 0.2)
@@
 	)
 	(via
-		(at 150.38 87.87)
+		(at 155.52 91.34)
 		(size 0.5)
 		(drill 0.2)
@@
 	)
 	(via
-		(at 156.01 91.62)
+		(at 154.956667 94.55)
 		(size 0.5)
 		(drill 0.2)
@@
 	)
 	(via
+		(at 156.73 94.55)
+		(size 0.5)
+		(drill 0.2)
+		(layers "F.Cu" "B.Cu")
+		(free yes)
+		(net 1)
+	)
+	(via
 		(at 155.38 80.37)
 		(size 0.5)
@@
 	)
 	(via
+		(at 159.1 94.55)
+		(size 0.5)
+		(drill 0.2)
+		(layers "F.Cu" "B.Cu")
+		(free yes)
+		(net 1)
+	)
+	(via
+		(at 160.83 94.55)
+		(size 0.5)
+		(drill 0.2)
+		(layers "F.Cu" "B.Cu")
+		(free yes)
+		(net 1)
+	)
+	(via
 		(at 160.98 84.93)
 		(size 0.5)
@@
 	)
 	(segment
-		(start 156.97 93.55)
-		(end 159.68 96.26)
-		(width 0.4983)
+		(start 160.7625 96.26)
+		(end 159.990927 96.26)
+		(width 0.824573)
 		(layer "B.Cu")
 		(net 6)
 	)
 	(segment
-		(start 159.68 96.26)
-		(end 160.7625 96.26)
-		(width 0.4983)
+		(start 159.28382 95.967107)
+		(end 156.97 93.653287)
+		(width 0.824573)
+		(layer "B.Cu")
+		(net 6)
+	)
+	(arc
+		(start 159.990927 96.26)
+		(mid 159.608244 96.18388)
+		(end 159.28382 95.967107)
+		(width 0.824573)
 		(layer "B.Cu")
 		(net 6)
@@
 	)
 	(segment
-		(start 156.97 90.805)
-		(end 156.97 90.08)
-		(width 0.4983)
+		(start 156.97 90.08)
+		(end 156.97 90.805)
+		(width 0.2)
 		(layer "B.Cu")
 		(net 9)
@@
 		(start 156.97 91.445)
 		(end 156.97 92.18)
-		(width 0.4983)
+		(width 0.2)
 		(layer "B.Cu")
 		(net 11)
 	)
 	(segment
-		(start 156.97 92.18)
-		(end 156.97 92.91)
-		(width 0.4983)
+		(start 156.97 92.91)
+		(end 156.97 92.18)
+		(width 0.2)
 		(layer "B.Cu")
 		(net 11)
@@
 		(placement
 			(enabled no)
-			(sheetname "")
+			(sheetname "/")
 		)
 		(fill
@@
 		(polygon
 			(pts
-				(xy 162 94.61) (xy 162 97.61) (xy 150 97.61) (xy 150 94.61)
+				(xy 162 97.61) (xy 162 94.91) (xy 150 94.91) (xy 150 97.61)
 			)
 		)
