File: pcb/dongle.kicad_sch (KiCad schematic)
At the start: 32 parts, among them J1 USB_A, J2 Conn_01x01_Pin, J3 Conn_01x01_Pin, J4 Conn_01x01_Pin, J5 Conn_01x01_Pin, SW1 SW_Push_45deg, U3 nRF52833_QDxx, Y1 32MHz

Commit message: update pcb
Parts:
- AE1: footprint (none) -> dongle:Texas_SWRA117D_2.4GHz_Left
- D1: footprint (none) -> dongle:LED_0603_1608Metric
- R1: footprint (none) -> dongle:R_0201_0603Metric_Pad0.64x0.40mm_HandSolder
- SW1: footprint (none) -> dongle:TS342A2P
Changed lines of the file:
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@@
 	)
 	(junction
+		(at 170.18 72.39)
+		(diameter 0)
+		(color 0 0 0 0)
+	)
+	(junction
 		(at 201.93 31.75)
 		(diameter 0)
@@
 	)
 	(junction
-		(at 170.18 71.12)
-		(diameter 0)
-		(color 0 0 0 0)
-	)
-	(junction
 		(at 114.3 92.71)
 		(diameter 0)
@@
 	(wire
 		(pts
+			(xy 170.18 72.39) (xy 170.18 73.66)
+		)
+		(stroke
+			(width 0)
+			(type default)
+		)
+	)
+	(wire
+		(pts
 			(xy 220.98 60.96) (xy 187.96 60.96)
 		)
@@
 	(wire
 		(pts
+			(xy 170.18 71.12) (xy 170.18 72.39)
+		)
+		(stroke
+			(width 0)
+			(type default)
+		)
+	)
+	(wire
+		(pts
 			(xy 219.71 39.37) (xy 215.9 39.37)
 		)
@@
 	(wire
 		(pts
+			(xy 176.53 72.39) (xy 170.18 72.39)
+		)
+		(stroke
+			(width 0)
+			(type default)
+		)
+	)
+	(wire
+		(pts
 			(xy 251.46 63.5) (xy 247.65 63.5)
 		)
@@
 	(wire
 		(pts
-			(xy 273.05 63.5) (xy 269.24 63.5)
+			(xy 59.69 177.8) (xy 62.23 177.8)
 		)
 		(stroke
@@
 	(wire
 		(pts
-			(xy 252.73 21.59) (xy 252.73 30.48)
+			(xy 273.05 63.5) (xy 269.24 63.5)
 		)
 		(stroke
@@
 	(wire
 		(pts
-			(xy 176.53 71.12) (xy 170.18 71.12)
+			(xy 252.73 21.59) (xy 252.73 30.48)
 		)
 		(stroke
@@
 		)
 	)
-	(global_label "VSS"
+	(global_label "D+"
 		(shape input)
-		(at 176.53 71.12 0)
+		(at 130.81 31.75 0)
 		(fields_autoplaced yes)
 		(effects
@@
 		)
 		(property "Intersheetrefs" "${INTERSHEET_REFS}"
-			(at 183.0228 71.12 0)
+			(at 136.6376 31.75 0)
 			(effects
 				(font
@@
 		)
 	)
-	(global_label "D+"
+	(global_label "DEC5"
 		(shape input)
-		(at 130.81 31.75 0)
+		(at 49.53 35.56 90)
 		(fields_autoplaced yes)
 		(effects
@@
 		)
 		(property "Intersheetrefs" "${INTERSHEET_REFS}"
-			(at 136.6376 31.75 0)
+			(at 49.53 27.6763 90)
 			(effects
 				(font
@@
 		)
 	)
-	(global_label "DEC5"
+	(global_label "DEC1"
 		(shape input)
-		(at 49.53 35.56 90)
+		(at 39.37 35.56 90)
 		(fields_autoplaced yes)
 		(effects
@@
 		)
 		(property "Intersheetrefs" "${INTERSHEET_REFS}"
-			(at 49.53 27.6763 90)
+			(at 39.37 27.6763 90)
 			(effects
 				(font
@@
 		)
 	)
-	(global_label "DEC1"
+	(global_label "ANT"
 		(shape input)
-		(at 39.37 35.56 90)
+		(at 219.71 31.75 0)
 		(fields_autoplaced yes)
 		(effects
@@
 		)
 		(property "Intersheetrefs" "${INTERSHEET_REFS}"
-			(at 39.37 27.6763 90)
+			(at 226.0819 31.75 0)
 			(effects
 				(font
@@
 		)
 	)
-	(global_label "ANT"
+	(global_label "VDD"
 		(shape input)
-		(at 219.71 31.75 0)
+		(at 59.69 35.56 90)
 		(fields_autoplaced yes)
 		(effects
@@
 		)
 		(property "Intersheetrefs" "${INTERSHEET_REFS}"
-			(at 226.0819 31.75 0)
+			(at 59.69 28.9462 90)
 			(effects
 				(font
@@
 		)
 	)
-	(global_label "VDD"
+	(global_label "VSS"
 		(shape input)
-		(at 59.69 35.56 90)
+		(at 176.53 72.39 0)
 		(fields_autoplaced yes)
 		(effects
@@
 		)
 		(property "Intersheetrefs" "${INTERSHEET_REFS}"
-			(at 59.69 28.9462 90)
+			(at 183.0228 72.39 0)
 			(effects
 				(font
@@
 		)
 	)
-	(global_label "VSS"
-		(shape input)
-		(at 59.69 177.8 270)
-		(fields_autoplaced yes)
-		(effects
-			(font
-				(size 1.27 1.27)
-			)
-			(justify right)
-		)
-		(property "Intersheetrefs" "${INTERSHEET_REFS}"
-			(at 59.69 184.2928 90)
-			(effects
-				(font
-					(size 1.27 1.27)
-				)
-				(justify right)
-				(hide yes)
-			)
-		)
-	)
 	(global_label "DEC1"
 		(shape input)
@@
 		)
 	)
+	(global_label "VSS"
+		(shape input)
+		(at 60.96 177.8 270)
+		(fields_autoplaced yes)
+		(effects
+			(font
+				(size 1.27 1.27)
+			)
+			(justify right)
+		)
+		(property "Intersheetrefs" "${INTERSHEET_REFS}"
+			(at 60.96 184.2928 90)
+			(effects
+				(font
+					(size 1.27 1.27)
+				)
+				(justify right)
+				(hide yes)
+			)
+		)
+	)
 	(global_label "VDD"
 		(shape input)
@@
 		)
 	)
-	(global_label "VSS_PA"
-		(shape input)
-		(at 62.23 177.8 270)
-		(fields_autoplaced yes)
-		(effects
-			(font
-				(size 1.27 1.27)
-			)
-			(justify right)
-		)
-		(property "Intersheetrefs" "${INTERSHEET_REFS}"
-			(at 62.23 187.619 90)
-			(effects
-				(font
-					(size 1.27 1.27)
-				)
-				(justify right)
-				(hide yes)
-			)
-		)
-	)
 	(global_label "DEC6"
 		(shape input)
@@
 			)
 		)
-		(property "Footprint" ""
+		(property "Footprint" "dongle:TS342A2P"
 			(at 259.08 86.36 0)
 			(effects
@@
 	(symbol
 		(lib_id "Library:GND")
-		(at 170.18 71.12 0)
+		(at 170.18 73.66 0)
 		(unit 1)
 		(exclude_from_sim no)
@@
 		(fields_autoplaced yes)
 		(property "Reference" "#PWR07"
-			(at 170.18 77.47 0)
+			(at 170.18 80.01 0)
 			(effects
 				(font
@@
 		)
 		(property "Value" "GND"
-			(at 170.18 76.2 0)
+			(at 170.18 78.74 0)
 			(effects
 				(font
@@
 		)
 		(property "Footprint" ""
-			(at 170.18 71.12 0)
+			(at 170.18 73.66 0)
 			(effects
 				(font
@@
 		)
 		(property "Datasheet" ""
-			(at 170.18 71.12 0)
+			(at 170.18 73.66 0)
 			(effects
 				(font
@@
 		)
 		(property "Description" "Global ground symbol"
-			(at 170.18 80.518 0)
+			(at 170.18 83.058 0)
 			(effects
 				(font
@@
 			)
 		)
-		(property "Footprint" ""
+		(property "Footprint" "dongle:Texas_SWRA117D_2.4GHz_Left"
 			(at 187.96 26.67 0)
 			(effects
@@
 			)
 		)
-		(property "Footprint" ""
+		(property "Footprint" "dongle:R_0201_0603Metric_Pad0.64x0.40mm_HandSolder"
 			(at 265.43 65.278 90)
 			(effects
@@
 			)
 		)
-		(property "Footprint" ""
+		(property "Footprint" "dongle:LED_0603_1608Metric"
 			(at 255.27 63.5 0)
 			(effects

Commit message: update pcb
Parts:
- removed AE1: Antenna, dongle:Texas_SWRA117D_2.4GHz_Left, symbol dongle:Antenna
- removed Y1: 32MHz, dongle:Crystal_SMD_2012-2Pin_2.0x1.2mm_HandSoldering, symbol PNCATEHO_lowair:Crystal
- added AE1: Antenna_Shield, dongle:ANTC5020X110N, symbol dongle:Antenna_Shield
- added Y1: Crystal_GND24, dongle:Crystal_SMD_3225-4Pin_3.2x2.5mm, symbol dongle:Crystal_GND24
- C1, C10, C11, C2, C3, C4, C5, C7: footprint dongle:C_0201_0603Metric_Pad0.64x0.40mm_HandSolder -> dongle:C_0201_0603Metric
- C12, C13: footprint dongle:C_0402_1005Metric_Pad0.74x0.62mm_HandSolder -> dongle:C_0402_1005Metric
- C17, C19, C6: footprint dongle:C_0603_1608Metric_Pad1.08x0.95mm_HandSolder -> dongle:C_0603_1608Metric
- D1: footprint dongle:LED_0603_1608Metric -> dongle:LED_0402_1005Metric
- J2, J3, J4: footprint dongle:TestPoint_Pad_1.0x1.0mm -> dongle:TestPoint_Pad_D1.0mm
- J5: footprint dongle:TestPoint_Pad_D1.0mm -> dongle:TestPoint_Pad_1.0x1.0mm
- L1, L2: footprint dongle:L_0201_0603Metric_Pad0.64x0.40mm_HandSolder -> dongle:L_0201_0603Metric
- R1: footprint dongle:R_0201_0603Metric_Pad0.64x0.40mm_HandSolder -> dongle:R_0402_1005Metric
Connections:
- net GND: now also C1.1, Y1.2, Y1.4; no longer C1.2
- net XC1: now also C1.2, Y1.1; no longer C2.2
- net XC2: now also C2.2, Y1.3; no longer C1.1
- net at L2.2: now also AE1.2 (Shield)
- no-connect marks 15 -> 16
Other:
- moved on the sheet: C1, C2

Commit message: udpate footprint
Parts:
- added Y2: Crystal_Small, dongle:Crystal_SMD_3215-2Pin_3.2x1.5mm, symbol dongle:Crystal_Small
- AE1: footprint dongle:ANTC5020X110N -> dongle:AN9520-245
- C15, C16: value 12pF -> 7pF; footprint dongle:C_0201_0603Metric_Pad0.64x0.40mm_HandSolder -> dongle:C_0201_0603Metric; now fitted; now in the parts list
- Y1: footprint dongle:Crystal_SMD_3225-4Pin_3.2x2.5mm -> dongle:Crystal_SMD_2520-4Pin_2.5x2.0mm
Connections:
- net GND: now also C15.2, C16.1
- net XL1: now also C16.2, Y2.2
- net XL2: now also C15.1, Y2.1
Other:
- moved on the sheet: C1, C2, Y1

Commit message: upload v0.1
Parts:
- J1: footprint dongle:USB_A_Connfly_DS1098_Horizontal -> dongle:USB_A_Molex_48037-2200_Horizontal
- SW1: footprint dongle:TS342A2P -> dongle:SW_SPST_B3U-1000P
Connections:
- net at L2.2: now also AE1.1 (A); no longer AE1.2 (Shield)
Other:
- moved on the sheet: AE1
Changed lines of the file:
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@@
 	)
 	(no_connect
-		(at 92.71 71.12)
+		(at 185.42 31.75)
 	)
 	(no_connect
-		(at 185.42 31.75)
+		(at 92.71 71.12)
 	)
 	(no_connect
@@
 			)
 		)
-		(property "Footprint" "dongle:TS342A2P"
+		(property "Footprint" "dongle:SW_SPST_B3U-1000P"
 			(at 259.08 86.36 0)
 			(effects
@@
 			)
 		)
-		(property "Footprint" "dongle:USB_A_Connfly_DS1098_Horizontal"
+		(property "Footprint" "dongle:USB_A_Molex_48037-2200_Horizontal"
 			(at 127 33.02 0)
 			(effects
@@
 	(symbol
 		(lib_id "dongle:Antenna_Shield")
-		(at 185.42 26.67 0)
+		(at 187.96 26.67 0)
+		(mirror y)
 		(unit 1)
 		(exclude_from_sim no)
@@
 		(dnp no)
 		(property "Reference" "AE1"
-			(at 187.706 20.828 0)
+			(at 186.436 17.78 0)
 			(effects
 				(font
 					(size 1.27 1.27)
 				)
-				(justify left)
+				(justify right)
 			)
 		)
 		(property "Value" "Antenna_Shield"
-			(at 187.706 23.368 0)
+			(at 186.436 20.32 0)
 			(effects
 				(font
 					(size 1.27 1.27)
 				)
-				(justify left)
+				(justify right)
 			)
 		)
 		(property "Footprint" "dongle:AN9520-245"
-			(at 185.42 24.13 0)
+			(at 187.96 24.13 0)
 			(effects
 				(font
@@
 		)
 		(property "Datasheet" "~"
-			(at 185.42 24.13 0)
+			(at 187.96 24.13 0)
 			(effects
 				(font
@@
 		)
 		(property "Description" "Antenna with extra pin for shielding"
-			(at 185.42 26.67 0)
+			(at 187.96 26.67 0)
 			(effects
 				(font

Commit message: clear pcb
Connections:
- net GND: no longer C3.1, U3.25 (VSS_PA)
- new net VSS_PA: C3.1, U3.25 (VSS_PA)
Changed lines of the file:
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@@
-	)
-	(junction
-		(at 170.18 72.39)
-		(diameter 0)
-		(color 0 0 0 0)
 	)
 	(junction
@@
 	)
 	(junction
-		(at 213.36 77.47)
-		(diameter 0)
-		(color 0 0 0 0)
-	)
-	(junction
 		(at 123.19 43.18)
 		(diameter 0)
@@
 		(color 0 0 0 0)
 	)
-	(junction
-		(at 215.9 39.37)
-		(diameter 0)
-		(color 0 0 0 0)
-	)
 	(no_connect
 		(at 92.71 147.32)
@@
 	(wire
 		(pts
-			(xy 179.07 63.5) (xy 170.18 63.5)
-		)
-		(stroke
-			(width 0)
-			(type default)
-		)
-	)
-	(wire
-		(pts
-			(xy 222.25 77.47) (xy 213.36 77.47)
+			(xy 176.53 63.5) (xy 170.18 63.5)
 		)
 		(stroke
@@
 	(wire
 		(pts
-			(xy 170.18 72.39) (xy 170.18 73.66)
+			(xy 170.18 71.12) (xy 170.18 72.39)
 		)
 		(stroke
@@
 	(wire
 		(pts
-			(xy 170.18 71.12) (xy 170.18 72.39)
-		)
-		(stroke
-			(width 0)
-			(type default)
-		)
-	)
-	(wire
-		(pts
-			(xy 219.71 39.37) (xy 215.9 39.37)
+			(xy 218.44 39.37) (xy 215.9 39.37)
 		)
 		(stroke
@@
 	(wire
 		(pts
-			(xy 176.53 72.39) (xy 170.18 72.39)
-		)
-		(stroke
-			(width 0)
-			(type default)
-		)
-	)
-	(wire
-		(pts
 			(xy 251.46 63.5) (xy 247.65 63.5)
 		)
@@
 		)
 	)
-	(global_label "VSS"
-		(shape input)
-		(at 176.53 72.39 0)
-		(fields_autoplaced yes)
-		(effects
-			(font
-				(size 1.27 1.27)
-			)
-			(justify left)
-		)
-		(property "Intersheetrefs" "${INTERSHEET_REFS}"
-			(at 183.0228 72.39 0)
-			(effects
-				(font
-					(size 1.27 1.27)
-				)
-				(justify left)
-				(hide yes)
-			)
-		)
-	)
 	(global_label "VDD"
 		(shape input)
-		(at 179.07 63.5 0)
-		(fields_autoplaced yes)
-		(effects
-			(font
-				(size 1.27 1.27)
-			)
-			(justify left)
-		)
-		(property "Intersheetrefs" "${INTERSHEET_REFS}"
-			(at 185.6838 63.5 0)
+		(at 176.53 63.5 0)
+		(fields_autoplaced yes)
+		(effects
+			(font
+				(size 1.27 1.27)
+			)
+			(justify left)
+		)
+		(property "Intersheetrefs" "${INTERSHEET_REFS}"
+			(at 183.1438 63.5 0)
 			(effects
 				(font
@@
 		)
 	)
-	(global_label "VSS"
-		(shape input)
-		(at 222.25 77.47 0)
-		(fields_autoplaced yes)
-		(effects
-			(font
-				(size 1.27 1.27)
-			)
-			(justify left)
-		)
-		(property "Intersheetrefs" "${INTERSHEET_REFS}"
-			(at 228.7428 77.47 0)
-			(effects
-				(font
-					(size 1.27 1.27)
-				)
-				(justify left)
-				(hide yes)
-			)
-		)
-	)
 	(global_label "VBUS"
 		(shape input)
@@
 	(global_label "VSS_PA"
 		(shape input)
-		(at 219.71 39.37 0)
-		(fields_autoplaced yes)
-		(effects
-			(font
-				(size 1.27 1.27)
-			)
-			(justify left)
-		)
-		(property "Intersheetrefs" "${INTERSHEET_REFS}"
-			(at 229.529 39.37 0)
+		(at 218.44 39.37 0)
+		(fields_autoplaced yes)
+		(effects
+			(font
+				(size 1.27 1.27)
+			)
+			(justify left)
+		)
+		(property "Intersheetrefs" "${INTERSHEET_REFS}"
+			(at 228.259 39.37 0)
 			(effects
 				(font
@@
 				)
 				(justify left)
-				(hide yes)
-			)
-		)
-	)
-	(global_label "VSS"
-		(shape input)
-		(at 59.69 177.8 270)
-		(fields_autoplaced yes)
-		(effects
-			(font
-				(size 1.27 1.27)
-			)
-			(justify right)
-		)
-		(property "Intersheetrefs" "${INTERSHEET_REFS}"
-			(at 59.69 184.2928 90)
-			(effects
-				(font
-					(size 1.27 1.27)
-				)
-				(justify right)
 				(hide yes)
 			)
@@
 				(path "/81b8789c-509b-48aa-aabd-6327c54a25df"
 					(reference "J5")
-					(unit 1)
-				)
-			)
-		)
-	)
-	(symbol
-		(lib_id "PNCATEHO_lowair:GND")
-		(at 215.9 39.37 0)
-		(mirror y)
-		(unit 1)
-		(exclude_from_sim no)
-		(in_bom yes)
-		(on_board yes)
-		(dnp no)
-		(fields_autoplaced yes)
-		(property "Reference" "#PWR028"
-			(at 215.9 45.72 0)
-			(effects
-				(font
-					(size 1.27 1.27)
-				)
-				(hide yes)
-			)
-		)
-		(property "Value" "GND"
-			(at 215.9 44.45 0)
-			(effects
-				(font
-					(size 1.27 1.27)
-				)
-			)
-		)
-		(property "Footprint" ""
-			(at 215.9 39.37 0)
-			(effects
-				(font
-					(size 1.27 1.27)
-				)
-				(hide yes)
-			)
-		)
-		(property "Datasheet" ""
-			(at 215.9 39.37 0)
-			(effects
-				(font
-					(size 1.27 1.27)
-				)
-				(hide yes)
-			)
-		)
-		(property "Description" "Power symbol creates a global label with name \"GND\" , ground"
-			(at 215.9 39.37 0)
-			(effects
-				(font
-					(size 1.27 1.27)
-				)
-				(hide yes)
-			)
-		)
-		(pin "1"
-		)
-		(instances
-			(project "PNCATEHO_lowair"
-				(path "/81b8789c-509b-48aa-aabd-6327c54a25df"
-					(reference "#PWR028")
 					(unit 1)
 				)
@@
 	)
 	(symbol
+		(lib_id "Library:GND")
+		(at 59.69 177.8 0)
+		(unit 1)
+		(exclude_from_sim no)
+		(in_bom yes)
+		(on_board yes)
+		(dnp no)
+		(fields_autoplaced yes)
+		(property "Reference" "#PWR015"
+			(at 59.69 184.15 0)
+			(effects
+				(font
+					(size 1.27 1.27)
+				)
+				(hide yes)
+			)
+		)
+		(property "Value" "GND"
+			(at 59.69 182.88 0)
+			(effects
+				(font
+					(size 1.27 1.27)
+				)
+			)
+		)
+		(property "Footprint" ""
+			(at 59.69 177.8 0)
+			(effects
+				(font
+					(size 1.27 1.27)
+				)
+				(hide yes)
+			)
+		)
+		(property "Datasheet" ""
+			(at 59.69 177.8 0)
+			(effects
+				(font
+					(size 1.27 1.27)
+				)
+				(hide yes)
+			)
+		)
+		(property "Description" "Global ground symbol"
+			(at 59.69 187.198 0)
+			(effects
+				(font
+					(size 1.27 1.27)
+				)
+				(hide yes)
+			)
+		)
+		(pin "1"
+		)
+		(instances
+			(project "dongle"
+				(path "/81b8789c-509b-48aa-aabd-6327c54a25df"
+					(reference "#PWR015")
+					(unit 1)
+				)
+			)
+		)
+	)
+	(symbol
 		(lib_id "dongle:SW_Push_45deg")
 		(at 259.08 86.36 0)
@@
 	(symbol
 		(lib_id "Library:GND")
-		(at 170.18 73.66 0)
+		(at 170.18 72.39 0)
 		(unit 1)
 		(exclude_from_sim no)
@@
 		(fields_autoplaced yes)
 		(property "Reference" "#PWR07"
-			(at 170.18 80.01 0)
+			(at 170.18 78.74 0)
 			(effects
 				(font
@@
 		)
 		(property "Value" "GND"
-			(at 170.18 78.74 0)
+			(at 170.18 77.47 0)
 			(effects
 				(font
@@
 		)
 		(property "Footprint" ""
-			(at 170.18 73.66 0)
+			(at 170.18 72.39 0)
 			(effects
 				(font
@@
 		)
 		(property "Datasheet" ""
-			(at 170.18 73.66 0)
+			(at 170.18 72.39 0)
 			(effects
 				(font
@@
 		)
 		(property "Description" "Global ground symbol"
-			(at 170.18 83.058 0)
-			(effects
-				(font
+			(at 170.18 81.788 0)
+			(effects
+				(font

Commit message: update pcb
Connections:
- net GND: no longer C9.1
- net DEC4 renamed DEC4_6
- net DEC4_6: now also U3.26 (DEC6)
- net DEC5: no longer names the net of U3.21 (DEC5)
- net DEC6: no longer names the net of C9.2
- net DEC6: no longer U3.26 (DEC6)
- no-connect marks 16 -> 17
Other:
- moved on the sheet: C10, C13, C9
Changed lines of the file:
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@@
 	)
 	(junction
+		(at 203.2 74.93)
+		(diameter 0)
+		(color 0 0 0 0)
+	)
+	(junction
 		(at 123.19 43.18)
 		(diameter 0)
@@
 	)
 	(junction
-		(at 201.93 77.47)
-		(diameter 0)
-		(color 0 0 0 0)
-	)
-	(junction
 		(at 257.81 29.21)
 		(diameter 0)
@@
 	)
 	(no_connect
+		(at 49.53 35.56)
+	)
+	(no_connect
 		(at 92.71 48.26)
 	)
@@
 	(wire
 		(pts
-			(xy 220.98 60.96) (xy 187.96 60.96)
+			(xy 199.39 63.5) (xy 194.31 63.5)
 		)
 		(stroke
@@
 	(wire
 		(pts
-			(xy 220.98 66.04) (xy 201.93 66.04)
-		)
-		(stroke
-			(width 0)
-			(type default)
-		)
-	)
-	(wire
-		(pts
 			(xy 245.11 25.4) (xy 252.73 25.4)
 		)
@@
 	(wire
 		(pts
-			(xy 220.98 69.85) (xy 213.36 69.85)
+			(xy 213.36 67.31) (xy 210.82 67.31)
 		)
 		(stroke
@@
 	(wire
 		(pts
-			(xy 187.96 77.47) (xy 201.93 77.47)
+			(xy 194.31 74.93) (xy 203.2 74.93)
 		)
 		(stroke
@@
 	(wire
 		(pts
-			(xy 187.96 60.96) (xy 187.96 69.85)
+			(xy 194.31 63.5) (xy 194.31 67.31)
 		)
 		(stroke
@@
 	(wire
 		(pts
-			(xy 201.93 80.01) (xy 201.93 77.47)
+			(xy 203.2 77.47) (xy 203.2 74.93)
 		)
 		(stroke
@@
 	(wire
 		(pts
-			(xy 201.93 66.04) (xy 201.93 69.85)
+			(xy 255.27 41.91) (xy 255.27 44.45)
 		)
 		(stroke
@@
 	(wire
 		(pts
-			(xy 255.27 41.91) (xy 255.27 44.45)
+			(xy 64.77 27.94) (xy 64.77 35.56)
 		)
 		(stroke
@@
 	(wire
 		(pts
-			(xy 64.77 27.94) (xy 64.77 35.56)
+			(xy 114.3 60.96) (xy 114.3 63.5)
 		)
 		(stroke
@@
 	(wire
 		(pts
-			(xy 114.3 60.96) (xy 114.3 63.5)
+			(xy 251.46 63.5) (xy 247.65 63.5)
 		)
 		(stroke
@@
 	(wire
 		(pts
-			(xy 251.46 63.5) (xy 247.65 63.5)
+			(xy 245.11 25.4) (xy 245.11 29.21)
 		)
 		(stroke
@@
 	(wire
 		(pts
-			(xy 245.11 25.4) (xy 245.11 29.21)
+			(xy 203.2 74.93) (xy 210.82 74.93)
 		)
 		(stroke
@@
 	(wire
 		(pts
-			(xy 201.93 77.47) (xy 213.36 77.47)
-		)
-		(stroke
-			(width 0)
-			(type default)
-		)
-	)
-	(wire
-		(pts
 			(xy 245.11 21.59) (xy 245.11 25.4)
 		)
@@
 		)
 	)
-	(global_label "DEC5"
-		(shape input)
-		(at 49.53 35.56 90)
-		(fields_autoplaced yes)
-		(effects
-			(font
-				(size 1.27 1.27)
-			)
-			(justify left)
-		)
-		(property "Intersheetrefs" "${INTERSHEET_REFS}"
-			(at 49.53 27.6763 90)
-			(effects
-				(font
-					(size 1.27 1.27)
-				)
-				(justify left)
-				(hide yes)
-			)
-		)
-	)
 	(global_label "DEC1"
 		(shape input)
@@
 		)
 	)
-	(global_label "DEC6"
-		(shape input)
-		(at 220.98 66.04 0)
-		(fields_autoplaced yes)
-		(effects
-			(font
-				(size 1.27 1.27)
-			)
-			(justify left)
-		)
-		(property "Intersheetrefs" "${INTERSHEET_REFS}"
-			(at 228.8637 66.04 0)
-			(effects
-				(font
-					(size 1.27 1.27)
-				)
-				(justify left)
-				(hide yes)
-			)
-		)
-	)
 	(global_label "LED"
 		(shape input)
@@
 	(global_label "DEC3"
 		(shape input)
-		(at 220.98 60.96 0)
+		(at 199.39 63.5 0)
 		(fields_autoplaced yes)
 		(effects
@@
 		)
 		(property "Intersheetrefs" "${INTERSHEET_REFS}"
-			(at 228.8637 60.96 0)
+			(at 207.2737 63.5 0)
 			(effects
 				(font
@@
 		)
 	)
-	(global_label "DEC4"
+	(global_label "DEC4_6"
 		(shape input)
 		(at 46.99 35.56 90)
@@
 		)
 		(property "Intersheetrefs" "${INTERSHEET_REFS}"
-			(at 46.99 27.6763 90)
+			(at 46.99 25.4992 90)
+			(effects
+				(font
+					(size 1.27 1.27)
+				)
+				(justify left)
+				(hide yes)
+			)
+		)
+	)
+	(global_label "DEC4_6"
+		(shape input)
+		(at 213.36 67.31 0)
+		(fields_autoplaced yes)
+		(effects
+			(font
+				(size 1.27 1.27)
+			)
+			(justify left)
+		)
+		(property "Intersheetrefs" "${INTERSHEET_REFS}"
+			(at 223.4208 67.31 0)
 			(effects
 				(font
@@
 		)
 	)
-	(global_label "DEC6"
+	(global_label "DEC4_6"
 		(shape input)
 		(at 52.07 35.56 90)
@@
 		)
 		(property "Intersheetrefs" "${INTERSHEET_REFS}"
-			(at 52.07 27.6763 90)
+			(at 52.07 25.4992 90)
 			(effects
 				(font
@@
 		)
 	)
-	(global_label "DEC4"
-		(shape input)
-		(at 220.98 69.85 0)
-		(fields_autoplaced yes)
-		(effects
-			(font
-				(size 1.27 1.27)
-			)
-			(justify left)
-		)
-		(property "Intersheetrefs" "${INTERSHEET_REFS}"
-			(at 228.8637 69.85 0)
-			(effects
-				(font
-					(size 1.27 1.27)
-				)
-				(justify left)
-				(hide yes)
-			)
-		)
-	)
 	(global_label "SWD"
 		(shape input)
@@
 	(symbol
 		(lib_id "Library:GND")
-		(at 201.93 80.01 0)
+		(at 203.2 77.47 0)
 		(unit 1)
 		(exclude_from_sim no)
@@
 		(fields_autoplaced yes)
 		(property "Reference" "#PWR08"
-			(at 201.93 86.36 0)
+			(at 203.2 83.82 0)
 			(effects
 				(font
@@
 		)
 		(property "Value" "GND"
-			(at 201.93 85.09 0)
+			(at 203.2 82.55 0)
 			(effects
 				(font
@@
 		)
 		(property "Footprint" ""
-			(at 201.93 80.01 0)
+			(at 203.2 77.47 0)
 			(effects
 				(font
@@
 		)
 		(property "Datasheet" ""
-			(at 201.93 80.01 0)
+			(at 203.2 77.47 0)
 			(effects
 				(font
@@
 		)
 		(property "Description" "Global ground symbol"
-			(at 201.93 89.408 0)
+			(at 203.2 86.868 0)
 			(effects
 				(font
@@
 	(symbol
 		(lib_id "PNCATEHO_lowair:C")
-		(at 187.96 73.66 0)
+		(at 194.31 71.12 0)
 		(mirror x)
 		(unit 1)
@@
 		(dnp no)
 		(property "Reference" "C10"
-			(at 191.262 74.93 0)
+			(at 197.612 72.39 0)
 			(effects
 				(font
@@
 		)
 		(property "Value" "100pF"
-			(at 191.262 72.39 0)
+			(at 197.612 69.85 0)
 			(effects
 				(font
@@
 		)
 		(property "Footprint" "dongle:C_0201_0603Metric"
-			(at 188.9252 69.85 0)
+			(at 195.2752 67.31 0)
 			(effects
 				(font
@@
 		)
 		(property "Datasheet" "~"
-			(at 187.96 73.66 0)
+			(at 194.31 71.12 0)
 			(effects
 				(font
@@
 		)
 		(property "Description" "Unpolarized capacitor"
-			(at 187.96 73.66 0)
+			(at 194.31 71.12 0)
 			(effects
 				(font
@@
 	(symbol
 		(lib_id "PNCATEHO_lowair:C")
-		(at 213.36 73.66 0)
+		(at 210.82 71.12 0)
 		(mirror x)
 		(unit 1)
@@
 		(dnp no)
 		(property "Reference" "C13"
-			(at 216.408 74.93 0)
+			(at 213.868 72.39 0)
 			(effects
 				(font
@@
 		)
 		(property "Value" "1uF"
-			(at 216.408 72.39 0)
+			(at 213.868 69.85 0)
 			(effects
 				(font
@@
 		)
 		(property "Footprint" "dongle:C_0402_1005Metric"
-			(at 214.3252 69.85 0)
+			(at 211.7852 67.31 0)
 			(effects
 				(font
@@
 		)
 		(property "Datasheet" "~"
-			(at 213.36 73.66 0)
+			(at 210.82 71.12 0)
 			(effects
 				(font
@@
 		)
 		(property "Description" "Unpolarized capacitor"
-			(at 213.36 73.66 0)
+			(at 210.82 71.12 0)
 			(effects
 				(font
@@
 	(symbol
 		(lib_id "PNCATEHO_lowair:C")
-		(at 201.93 73.66 0)
+		(at 180.34 100.33 0)
 		(mirror x)
 		(unit 1)
@@
 		(dnp yes)
 		(property "Reference" "C9"
-			(at 205.232 74.93 0)
+			(at 183.642 101.6 0)
 			(effects
 				(font
@@
 		)
 		(property "Value" "N.C"
-			(at 205.232 72.39 0)
+			(at 183.642 99.06 0)
 			(effects
 				(font
@@
 		)
 		(property "Footprint" "PNCATEHO_lowair:C_0201_0603Metric_Pad0.64x0.40mm_HandSolder"
-			(at 202.8952 69.85 0)
+			(at 181.3052 96.52 0)
 			(effects
 				(font
@@
 		)
 		(property "Datasheet" "~"
-			(at 201.93 73.66 0)
+			(at 180.34 100.33 0)
 			(effects
 				(font
@@
 		)
 		(property "Description" "Unpolarized capacitor"
-			(at 201.93 73.66 0)
+			(at 180.34 100.33 0)
 			(effects
 				(font
